File: stryfe_fuse_board.kicad_pcb (KiCad board)
At the start: 2 copper layers, 2 parts

Commit message: kicad updates
Parts:
- added J1: Screw_Terminal_01x02, donutbrary:Amass_XT60PW-M_Kombifootprint, F.Cu at (157.5, 71.1)
- added J2: Conn_01x02, donutbrary:Amass_XT60PW-M_Kombifootprint, F.Cu at (127.0, 71.1)
- moved F2 12.7 mm to (149.0, 66.2), turned to -90 degrees
- moved F1 10.4 mm to (136.0, 75.7), turned to 90 degrees
Routing:
- net Net-(J1-Pad2): track 0.00 -> 0.51 mm
- added copper zone on B.Cu, net GND
- added copper zone on F.Cu, net Net-(F1-Pad2)
- added copper zone on F.Cu, net Net-(J1-Pad2)
Other:
- board outline added: 55.9 x 22.9 mm
- rule pad_to_mask_clearance: 0 -> 0.05
