File: stryfe_fuse_board.kicad_sch (KiCad schematic)
At the start: 4 parts, among them J1 Screw_Terminal_01x02, J2 Conn_01x02

Commit message: kicad updates
Parts:
- J1: footprint TerminalBlock:TerminalBlock_Altech_AK300-2_P5.00mm -> donutbrary:Amass_XT60PW-M_Kombifootprint
- J2: footprint (none) -> donutbrary:Amass_XT60PW-M_Kombifootprint
Connections:
- net GND: now reaches J1.1 (Pin_1), J2.1 (Pin_1)
Changed lines of the file:
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@@
   (junction (at 99.695 85.09) (diameter 0) (color 0 0 0 0)
-  )
-  (wire (pts (xy 84.455 87.63) (xy 87.63 87.63))
-    (stroke (width 0) (type default) (color 0 0 0 0))
-  )
-  (wire (pts (xy 107.95 85.09) (xy 107.95 90.17))
-    (stroke (width 0) (type default) (color 0 0 0 0))
   )
   (wire (pts (xy 88.9 92.71) (xy 92.71 92.71))
     (stroke (width 0) (type default) (color 0 0 0 0))
   )
-  (wire (pts (xy 99.695 85.09) (xy 107.95 85.09))
-    (stroke (width 0) (type default) (color 0 0 0 0))
-  )
-  (wire (pts (xy 111.76 83.82) (xy 111.76 87.63))
+  (wire (pts (xy 99.695 85.09) (xy 111.76 85.09))
     (stroke (width 0) (type default) (color 0 0 0 0))
   )
@@
     (stroke (width 0) (type default) (color 0 0 0 0))
   )
-  (wire (pts (xy 107.95 90.17) (xy 111.76 90.17))
-    (stroke (width 0) (type default) (color 0 0 0 0))
-  )
-  (wire (pts (xy 87.63 83.82) (xy 111.76 83.82))
+  (wire (pts (xy 111.76 85.09) (xy 111.76 87.63))
     (stroke (width 0) (type default) (color 0 0 0 0))
   )
@@
     (stroke (width 0) (type default) (color 0 0 0 0))
   )
-  (wire (pts (xy 87.63 87.63) (xy 87.63 83.82))
-    (stroke (width 0) (type default) (color 0 0 0 0))
+  (symbol (lib_id "donutbrary:GND") (at 111.76 90.17 0) (unit 1)
+    (in_bom yes) (on_board yes) (fields_autoplaced)
+    (property "Reference" "#PWR?" (id 0) (at 111.76 96.52 0)
+      (effects (font (size 1.27 1.27)) hide)
+    )
+    (property "Value" "GND" (id 1) (at 111.76 94.7325 0))
+    (property "Footprint" "" (id 2) (at 111.76 90.17 0)
+      (effects (font (size 1.27 1.27)) hide)
+    )
+    (property "Datasheet" "" (id 3) (at 111.76 90.17 0)
+      (effects (font (size 1.27 1.27)) hide)
+    )
+    (pin "1")
+  )
+  (symbol (lib_id "donutbrary:GND") (at 84.455 87.63 0) (unit 1)
+    (in_bom yes) (on_board yes) (fields_autoplaced)
+    (property "Reference" "#PWR?" (id 0) (at 84.455 93.98 0)
+      (effects (font (size 1.27 1.27)) hide)
+    )
+    (property "Value" "GND" (id 1) (at 84.455 92.1925 0))
+    (property "Footprint" "" (id 2) (at 84.455 87.63 0)
+      (effects (font (size 1.27 1.27)) hide)
+    )
+    (property "Datasheet" "" (id 3) (at 84.455 87.63 0)
+      (effects (font (size 1.27 1.27)) hide)
+    )
+    (pin "1")
   )
   (symbol (lib_id "Device:Fuse") (at 92.71 88.9 0) (unit 1)
@@
     (property "Reference" "J2" (id 0) (at 79.375 82.3935 0))
     (property "Value" "Conn_01x02" (id 1) (at 79.375 85.1686 0))
-    (property "Footprint" "" (id 2) (at 79.375 87.63 0)
+    (property "Footprint" "donutbrary:Amass_XT60PW-M_Kombifootprint" (id 2) (at 79.375 87.63 0)
       (effects (font (size 1.27 1.27)) hide)
     )
@@
     (pin "2")
   )
-  (symbol (lib_id "Connector:Screw_Terminal_01x02") (at 116.84 87.63 0) (unit 1)
+  (symbol (lib_id "Connector:Screw_Terminal_01x02") (at 116.84 90.17 0) (mirror x) (unit 1)
     (in_bom yes) (on_board yes) (fields_autoplaced)
-    (property "Reference" "J1" (id 0) (at 118.872 87.9915 0)
-      (effects (font (size 1.27 1.27)) (justify left))
-    )
-    (property "Value" "Screw_Terminal_01x02" (id 1) (at 118.872 90.7666 0)
-      (effects (font (size 1.27 1.27)) (justify left))
-    )
-    (property "Footprint" "TerminalBlock:TerminalBlock_Altech_AK300-2_P5.00mm" (id 2) (at 116.84 87.63 0)
+    (property "Reference" "J1" (id 0) (at 116.84 82.3935 0))
+    (property "Value" "Screw_Terminal_01x02" (id 1) (at 116.84 85.1686 0))
+    (property "Footprint" "donutbrary:Amass_XT60PW-M_Kombifootprint" (id 2) (at 116.84 90.17 0)
       (effects (font (size 1.27 1.27)) hide)
     )
-    (property "Datasheet" "~" (id 3) (at 116.84 87.63 0)
+    (property "Datasheet" "~" (id 3) (at 116.84 90.17 0)
       (effects (font (size 1.27 1.27)) hide)
     )
@@
   )
   (symbol_instances
+    (path "/07f5fa33-1d5e-4b56-92e6-274f86b80cbf"
+      (reference "#PWR?") (unit 1) (value "GND") (footprint "")
+    )
+    (path "/13c4d8f9-8857-4b42-8989-8b650fe32b9f"
+      (reference "#PWR?") (unit 1) (value "GND") (footprint "")
+    )
     (path "/30e47b6e-9b81-4fd0-a84a-bb3f3829efe4"
       (reference "F1") (unit 1) (value "Fuse") (footprint "Fuse:Fuseholder_Blade_ATO_Littelfuse_Pudenz_2_Pin")
@@
     )
     (path "/a8cb4243-d9e2-484f-9920-fd39587cc71f"
-      (reference "J1") (unit 1) (value "Screw_Terminal_01x02") (footprint "TerminalBlock:TerminalBlock_Altech_AK300-2_P5.00mm")
+      (reference "J1") (unit 1) (value "Screw_Terminal_01x02") (footprint "donutbrary:Amass_XT60PW-M_Kombifootprint")
     )
     (path "/93d56d07-b0d6-4650-8ad8-cc1590e343a0"
-      (reference "J2") (unit 1) (value "Conn_01x02") (footprint "")
+      (reference "J2") (unit 1) (value "Conn_01x02") (footprint "donutbrary:Amass_XT60PW-M_Kombifootprint")
     )
   )
